Commit message: practising great

File: controlko_description/urdf/rrbot.urdf.xacro (robot description, xacro)
@@ -2,7 +2,10 @@
 <robot xmlns:xacro="http://wiki.ros.org/xacro" name="rrbot">
   <!-- Use this if parameters are set from the launch file, otherwise delete -->
-  <xacro:arg name="use_fake_hardware" default="false" />
-  <xacro:arg name="fake_sensor_commands" default="false" />
   <xacro:arg name="prefix" default="" />
+  <xacro:arg name="use_mock_hardware" default="false" />
+  <xacro:arg name="mock_sensor_commands" default="false" />
+  <xacro:arg name="sim_gazebo_classic" default="false" />
+  <xacro:arg name="sim_gazebo" default="false" />
+  <xacro:arg name="simulation_controllers" default="" />
   <xacro:include filename="$(find controlko_description)/urdf/rrbot/rrbot_macro.xacro"/>
   <xacro:include filename="$(find controlko_description)/urdf/rrbot/rrbot_macro.ros2_control.xacro"/>
@@ -17,5 +20,29 @@
     name="rrbot"
     prefix="$(arg prefix)"
-    use_fake_hardware="$(arg use_fake_hardware)"
-    fake_sensor_commands="$(arg fake_sensor_commands)" />
+    use_mock_hardware="$(arg use_mock_hardware)"
+    mock_sensor_commands="$(arg mock_sensor_commands)"
+    sim_gazebo_classic="$(arg sim_gazebo_classic)"
+    sim_gazebo="$(arg sim_gazebo)"/>
+   <!-- Add Gazebo Classic Plugins -->
+  <xacro:if value="$(arg sim_gazebo_classic)">
+    <!-- Gazebo plugins -->
+    <gazebo reference="world">
+    </gazebo>
+    <gazebo>
+      <plugin filename="libgazebo_ros2_control.so" name="gazebo_ros2_control">
+        <parameters>$(arg simulation_controllers)</parameters>
+      </plugin>
+    </gazebo>
+  </xacro:if>
+  <xacro:if value="$(arg sim_gazebo)">
+    <!-- Gazebo plugins -->
+    <gazebo reference="world">
+    </gazebo>
+    <gazebo>
+      <plugin filename="libign_ros2_control-system.so" name="ign_ros2_control::IgnitionROS2ControlPlugin">
+        <parameters>$(arg simulation_controllers)</parameters>
+        <controller_manager_node_name>$(arg prefix)controller_manager</controller_manager_node_name>
+      </plugin>
+    </gazebo>
+  </xacro:if>
 </robot>

File: controlko_description/urdf/rrbot/rrbot_macro.ros2_control.xacro (robot description, xacro)
@@ -1,14 +1,26 @@
 <?xml version="1.0" encoding="UTF-8"?>
 <robot xmlns:xacro="http://wiki.ros.org/xacro">
-  <xacro:macro name="rrbot_ros2_control" params="name prefix use_fake_hardware:=^|false fake_sensor_commands:=^|false">
+  <xacro:macro name="rrbot_ros2_control" params="
+               name
+               prefix
+               use_mock_hardware:=^|false
+               mock_sensor_commands:=^|false
+               sim_gazebo_classic:=^|false
+               sim_gazebo:=^|false">
     <ros2_control name="${name}" type="system">
       <hardware>
-        <xacro:if value="${use_fake_hardware}">
-          <plugin>fake_components/GenericSystem</plugin>
-          <param name="fake_sensor_commands">${fake_sensor_commands}</param>
-          <param name="state_following_offset">0.0</param>
+        <xacro:if value="${use_mock_hardware}">
+          <plugin>mock_components/GenericSystem</plugin>
+          <param name="mock_sensor_commands">${mock_sensor_commands}</param>
+          <!-- <param name="state_following_offset">0.0</param> -->
         </xacro:if>
-        <xacro:unless value="${use_fake_hardware}">
-          <plugin>robot_hardware_inteface/RobotHardwareInteface</plugin>
+        <xacro:if value="${sim_gazebo_classic}">
+          <plugin>gazebo_ros2_control/GazeboSystem</plugin>
+        </xacro:if>
+        <xacro:if value="${sim_gazebo}">
+          <plugin>ign_ros2_control/IgnitionSystem</plugin>
+        </xacro:if>
+        <xacro:unless value="${use_mock_hardware}">
+          <plugin>robot_hardware_interface/RobotHardwareInterface</plugin>
         </xacro:unless>
       </hardware>
@@ -33,44 +45,4 @@
         <param name="initial_position">0.0</param>
       </joint>
-      <joint name="${prefix}joint3">
-        <command_interface name="position">     <!-- Add/Remove interfaces as needed -->
-          <param name="min">-1</param>
-          <param name="max">1</param>
-        </command_interface>
-        <state_interface name="position"/>
-        <state_interface name="velocity"/>
-        <state_interface name="acceleration"/>
-        <param name="initial_position">0.0</param>
-      </joint>
-      <joint name="${prefix}joint4">
-        <command_interface name="position">     <!-- Add/Remove interfaces as needed -->
-          <param name="min">-1</param>
-          <param name="max">1</param>
-        </command_interface>
-        <state_interface name="position"/>
-        <state_interface name="velocity"/>
-        <state_interface name="acceleration"/>
-        <param name="initial_position">0.0</param>
-      </joint>
-      <joint name="${prefix}joint5">
-        <command_interface name="position">     <!-- Add/Remove interfaces as needed -->
-          <param name="min">-1</param>
-          <param name="max">1</param>
-        </command_interface>
-        <state_interface name="position"/>
-        <state_interface name="velocity"/>
-        <state_interface name="acceleration"/>
-        <param name="initial_position">0.0</param>
-      </joint>
-      <joint name="${prefix}joint6">
-        <command_interface name="position">     <!-- Add/Remove interfaces as needed -->
-          <param name="min">-1</param>
-          <param name="max">1</param>
-        </command_interface>
-        <state_interface name="position"/>
-        <state_interface name="velocity"/>
-        <state_interface name="acceleration"/>
-        <param name="initial_position">0.0</param>
-      </joint>
       <sensor name="tcp_fts_sensor">            <!-- Remove/change sensors as needed -->
         <state_interface name="fx"/>
@@ -81,5 +53,5 @@
         <state_interface name="tz"/>
         <param name="frame_id">tool0</param>    <!-- Change sensors as needed -->
-        <param name="min_fx">-100</param>
+        <!-- <param name="min_fx">-100</param>
         <param name="max_fx">100</param>
         <param name="min_fy">-100</param>
@@ -92,6 +64,14 @@
         <param name="max_ty">10</param>
         <param name="min_tz">-15</param>
-        <param name="max_tz">15</param>
-      </sensor>
+        <param name="max_tz">15</param> -->
+        </sensor>
+        <gpio name="flange_gpios">
+          <state_interface name="digital_in_1"/>
+          <state_interface name="digital_in_2"/>
+          <command_interface name="digital_out_1"/>
+          <state_interface name="digital_out_1"/>
+          <command_interface name="digital_out_2"/>
+          <state_interface name="digital_out_2"/>
+      </gpio>
     </ros2_control>
   </xacro:macro>

File: controlko_description/urdf/rrbot/rrbot_macro.xacro (robot description, xacro)
@@ -10,14 +10,14 @@
       <xacro:default_inertial/>
       <visual>
-        <origin rpy="0 0 0" xyz="0 0 0" />
+        <origin xyz="0 0 0.15" rpy="0 0 0"/>
         <geometry>
-          <cylinder length="0.3" radius="0.3" />
+          <box size="0.3 0.3 0.3" />
 <!--           <mesh filename="package://controlko_description/meshes/rrbot/visual/base_link.dae" /> -->
         </geometry>
       </visual>
       <collision>
-        <origin rpy="0 0 0" xyz="0 0 0" />
+        <origin xyz="0 0 0.15" rpy="0 0 0" />
         <geometry>
-          <cylinder length="0.3" radius="0.3" />
+          <box size="0.3 0.3 0.3" />
 <!--           <mesh filename="package://controlko_description/meshes/rrbot/collision/base_link.stl" /> -->
         </geometry>
@@ -30,14 +30,14 @@
       <xacro:default_inertial/>
       <visual>
-        <origin xyz="0 0 0" rpy="0 0 0" />
+        <origin xyz="0 0 0.25" rpy="0 0 0" />
         <geometry>
-          <cylinder length="0.3" radius="0.15" />
+          <cylinder length="0.5" radius="0.1" />
 <!--           <mesh filename="package://controlko_description/meshes/rrbot/visual/link1.dae" /> -->
         </geometry>
       </visual>
       <collision>
-        <origin xyz="0 0 0" rpy="0 0 0" />
+        <origin xyz="0 0 0.25" rpy="0 0 0" />
         <geometry>
-          <cylinder length="0.3" radius="0.15" />
+          <cylinder length="0.5" radius="0.1" />
 <!--           <mesh filename="package://controlko_description/meshes/rrbot/collision/link1.stl" /> -->
         </geometry>
@@ -50,110 +50,21 @@
       <xacro:default_inertial/>
       <visual>
-        <origin xyz="0 0 0" rpy="0 0 0" />
+        <origin xyz="0 0 0.3" rpy="0 0 0" />
         <geometry>
-          <cylinder length="0.8" radius="0.15" />
+          <box size="0.1 0.1 0.6" />
 <!--           <mesh filename="package://controlko_description/meshes/rrbot/visual/link2.dae" /> -->
         </geometry>
       </visual>
       <collision>
-        <origin xyz="0 0 0" rpy="0 0 0" />
+        <origin xyz="0 0 0.3" rpy="0 0 0" />
         <geometry>
-          <cylinder length="0.8" radius="0.15" />
+          <box size="0.1 0.1 0.6" />
 <!--           <mesh filename="package://controlko_description/meshes/rrbot/collision/link2.stl"  /> -->
         </geometry>
       </collision>
     </link>
-    <!-- link 3 -->
-    <link name="${prefix}link3">
-      <!-- Default inertial for Gazebo/Ingnition - copy and edit block from 'common.xacro'
-           to get more realistic behaviour-->
-      <xacro:default_inertial/>
-      <visual>
-        <origin xyz="0 0 0" rpy="0 0 0" />
-        <geometry>
-          <cylinder length="0.5" radius="0.10" />
-<!--           <mesh filename="package://controlko_description/meshes/rrbot/visual/link3.dae" /> -->
-        </geometry>
-      </visual>
-      <collision>
-        <origin xyz="0 0 0" rpy="0 0 0" />
-        <geometry>
-          <cylinder length="0.5" radius="0.10" />
-<!--           <mesh filename="package://controlko_description/meshes/rrbot/collision/link3.stl"  /> -->
-        </geometry>
-      </collision>
-    </link>
-    <!-- link 4 -->
-    <link name="${prefix}link4">
-      <!-- Default inertial for Gazebo/Ingnition - copy and edit block from 'common.xacro'
-           to get more realistic behaviour-->
-      <xacro:default_inertial/>
-      <visual>
-        <origin xyz="0 0 0" rpy="0 0 0" />
-        <geometry>
-          <cylinder length="0.1" radius="0.2" />
-<!--           <mesh filename="package://controlko_description/meshes/rrbot/visual/link4.dae" /> -->
-        </geometry>
-      </visual>
-      <collision>
-        <origin xyz="0 0 0" rpy="0 0 0" />
-        <geometry>
-          <cylinder length="0.1" radius="0.2" />
-<!--           <mesh filename="package://controlko_description/meshes/rrbot/collision/link4.stl"  /> -->
-        </geometry>
-      </collision>
-    </link>
-    <!-- link 5 -->
-    <link name="${prefix}link5">
-      <!-- Default inertial for Gazebo/Ingnition - copy and edit block from 'common.xacro'
-           to get more realistic behaviour-->
-      <xacro:default_inertial/>
-      <visual>
-        <origin xyz="0 0 0" rpy="0 0 0" />
-        <geometry>
-          <cylinder length="0.2" radius="0.1" />
-<!--           <mesh filename="package://controlko_description/meshes/rrbot/visual/link5.dae" /> -->
-        </geometry>
-      </visual>
-      <collision>
-        <origin xyz="0 0 0" rpy="0 0 0" />
-        <geometry>
-          <cylinder length="0.2" radius="0.1" />
-<!--           <mesh filename="package://controlko_description/meshes/rrbot/collision/link5.stl" /> -->
-        </geometry>
-      </collision>
-    </link>
-    <!-- link 6 -->
-    <link name="${prefix}link6">
-      <!-- Default inertial for Gazebo/Ingnition - copy and edit block from 'common.xacro'
-           to get more realistic behaviour-->
-      <xacro:default_inertial/>
-      <visual>
-        <origin xyz="0 0 0" rpy="0 0 0" />
-        <geometry>
-          <cylinder length="0.05" radius="0.1" />
-<!--           <mesh filename="package://controlko_description/meshes/rrbot/visual/link6.dae" /> -->
-        </geometry>
-      </visual>
-      <collision>
-        <origin xyz="0 0 0" rpy="0 0 0" />
-        <geometry>
-          <cylinder length="0.05" radius="0.1" />
-<!--           <mesh filename="package://controlko_description/meshes/rrbot/collision/link6.stl" /> -->
-        </geometry>
-      </collision>
-    </link>
-    <!-- All-zero tool frame. This frame should correspond to the TOOL frame of the robot's controller.) -->
-    <link name="${prefix}tool0" />
-    <!-- tool link -->
-<!-- START Delete if not needed -->
-    <!-- Standard frames for industrial robots. Also useful for manipulators.
-         (ROS-I specs - https://wiki.ros.org/Industrial/Tutorials/WorkingWithRosIndustrialRobotSupportPackages#Standardised_links_.2F_frames)-->
-    <!-- This frame should correspond to the BASE coordinate system of robot's controller.) -->
+    <link name="${prefix}tool0"/>
     <link name="${prefix}base" />
-    <!-- Frame for mounting EEF models to a manipulator. x+ axis points forward (REP 103). -->
     <link name="${prefix}flange" />
-<!-- END Delete if not needed  -->
-    <!-- END LINKS -->
     <!-- JOINTS -->
     <!-- base_joint fixes base_link to the environment -->
@@ -165,57 +76,25 @@
     <!-- joint 1 -->
     <joint name="${prefix}joint1" type="revolute">
-      <origin xyz="0 0 0.3" rpy="${pi} 0 0" />
+      <origin xyz="0 0 0.3" rpy="0 0 0" />
       <parent link="${prefix}base_link" />
       <child link="${prefix}link1" />
       <axis xyz="0 0 1" />
-      <limit effort="0" lower="${radians(-180)}" upper="${radians(180)}" velocity="${radians(180)}" />
+      <limit effort="0" lower="${radians(-380)}" upper="${radians(380)}" velocity="${radians(180)}" />
     </joint>
     <!-- joint 2 -->
     <joint name="${prefix}joint2" type="revolute">
-      <origin xyz="0 0 0.3" rpy="${pi/2} 0 0" />
+      <origin xyz="0 0 0.5" rpy="0 -${pi/2} 0" />
       <parent link="${prefix}link1" />
       <child link="${prefix}link2" />
-      <axis xyz="0 0 1" />
-      <limit effort="0" lower="${radians(-180)}" upper="${radians(180)}" velocity="${radians(180)}" />
+      <axis xyz="0 1 0" />
+      <limit effort="0" lower="${radians(-60)}" upper="${radians(240)}" velocity="${radians(180)}" />
     </joint>
-    <!-- joint 3 -->
-    <joint name="${prefix}joint3" type="revolute">
-      <origin xyz="0.8 0 0" rpy="0 0 0" />
+    <!--tool frame - fixed frame -->
+    <joint name="${prefix}link2-tool0" type="fixed">
       <parent link="${prefix}link2" />
-      <child link="${prefix}link3" />
-      <axis xyz="0 0 1" />
-      <limit effort="0" lower="${radians(-90)}" upper="${radians(180)}" velocity="${radians(270)}" />
+      <child link="${prefix}tool0" />
+      <origin xyz="0 0 0.6" rpy="0 ${-pi} ${-pi/2}" />
     </joint>
-    <!-- joint 4 -->
-    <joint name="${prefix}joint4" type="revolute">
-      <origin xyz="0 0.1 0" rpy="0 ${-pi/2} 0" />
-      <parent link="${prefix}link3" />
-      <child link="${prefix}link4" />
-      <axis xyz="0 0 1" />
-      <limit effort="0" lower="${radians(-360)}" upper="${radians(360)}" velocity="${radians(360)}" />
-    </joint>
-    <!-- joint 5 -->
-    <joint name="${prefix}joint5" type="revolute">
-      <origin xyz="0 0 -0.1" rpy="0 ${pi/2} 0" />
-      <parent link="${prefix}link4" />
-      <child link="${prefix}link5" />
-      <axis xyz="0 0 1" />
-      <limit effort="0" lower="${radians(-120)}" upper="${radians(120)}" velocity="${radians(540)}" />
-    </joint>
-    <!-- joint 6 -->
-    <joint name="${prefix}joint6" type="revolute">
-      <origin xyz="0 0 0.1" rpy="0 ${-pi/2} 0" />
-      <parent link="${prefix}link5" />
-      <child link="${prefix}link6" />
-      <axis xyz="0 0 1" />
-      <limit effort="0" lower="${radians(-360)}" upper="${radians(360)}" velocity="${radians(720)}" />
-    </joint>
-    <!-- tool frame - fixed frame -->
-    <joint name="${prefix}joint6-tool0" type="fixed">
-      <parent link="${prefix}link6" />
-      <child link="${prefix}tool0" />
-      <origin xyz="0 0 -0.115" rpy="0 ${-pi} ${-pi/2}" />
-    </joint>
-    <!-- END JOINTS -->
+    <!-- END JOINTS-->
 <!-- START Delete if not needed -->
     <!-- Standard frames for industrial robots. Also useful for manipulators.
@@ -232,4 +111,33 @@
     </joint>
 <!-- END Delete if not needed  -->
+     <!-- Add Gazebo Classic Plugins -->
+    <gazebo>
+      <plugin name="joint_state_publisher" filename="libgazebo_ros_joint_state_publisher.so">
+        <update_rate>100</update_rate>
+      </plugin>
+    </gazebo>
+    <gazebo reference="${prefix}joint1">
+      <plugin name="gazebo_ros_control" filename="libgazebo_ros2_control.so">
+        <robotNamespace>/</robotNamespace>
+      </plugin>
+    </gazebo>
+    <gazebo reference="${prefix}joint2">
+      <plugin name="gazebo_ros_control" filename="libgazebo_ros2_control.so">
+        <robotNamespace>/</robotNamespace>
+      </plugin>
+    </gazebo>
+    <!-- Gazebo Classic physics -->
+    <gazebo>
+      <static>false</static>
+      <gravity>0 0 -9.81</gravity>
+    </gazebo>
+    <!-- Add Gazebo Sim (Ignition) Support -->
+    <gazebo>
+      <plugin name="ignition_ros2_control" filename="libignition_ros2_control-system.so">
+        <ros>
+          <namespace>/</namespace>
+        </ros>
+      </plugin>
+    </gazebo>
   </xacro:macro>
 </robot>
